File: wwavusbepp/KiCad/WWAVUSBEPP.kicad_pcb (KiCad board)
At the start: 4 copper layers, 36.8 x 40.8 mm, 66 parts, among them J1 USB_B, J2 Conn_01x26_Female, J3 Conn_01x06_Female, J4 Conn_01x04_Male, J5 Conn_01x02_Male, U1 CY7C68013-56LFC, U2 LT1762-3.3, U3 NCP302LSN45T1G, U4 FM24C64B, X1 24Mhz, t1 TestPoint, t10 TestPoint, t11 TestPoint, t12 TestPoint, t13 TestPoint, t14 TestPoint, t15 TestPoint, t16 TestPoint, t17 TestPoint, t18 TestPoint, t19 TestPoint, t20 TestPoint, t21 TestPoint, t22 TestPoint, t23 TestPoint, t24 TestPoint, t25 TestPoint, t26 TestPoint, t27 TestPoint, t28 TestPoint, t29 TestPoint, t30 TestPoint, t31 TestPoint, t32 TestPoint, t33 TestPoint, t34 TestPoint, t36 TestPoint, t7 TestPoint, t8 TestPoint, t9 TestPoint

Commit message: wwavusbepp: small tweaks, "diy" silkscreen
Signed-off-by: John McMaster <johndmcmaster@gmail.com>
Other:
- board text added: "diy-wwavusbepp v01 (it wasn't me)"
- board text removed: "wwavusbepp v01 (it wasn't me)"
Changed lines of the file:
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@@
-(kicad_pcb (version 20171130) (host pcbnew 5.0.2+dfsg1-1)
+(kicad_pcb (version 20171130) (host pcbnew 5.1.2-f72e74a~84~ubuntu16.04.1)
   (general
     (thickness 1.6)
@@
     (zone_45_only no)
     (trace_min 0.1524)
-    (segment_width 0.2)
-    (edge_width 0.05)
     (via_size 0.6858)
     (via_drill 0.3302)
@@
     (uvia_min_size 0.6858)
     (uvia_min_drill 0.3048)
+    (edge_width 0.05)
+    (segment_width 0.2)
     (pcb_text_width 0.3)
     (pcb_text_size 1.5 1.5)
@@
     (visible_elements FFFFFF7F)
     (pcbplotparams
-      (layerselection 0x010fc_ffffffff)
-      (usegerberextensions false)
+      (layerselection 0x010f0_ffffffff)
+      (usegerberextensions true)
       (usegerberattributes false)
       (usegerberadvancedattributes false)
@@
       (outputformat 1)
       (mirror false)
-      (drillshape 1)
+      (drillshape 0)
       (scaleselection 1)
-      (outputdirectory ""))
+      (outputdirectory "diy-wwavusbepp_r1"))
   )
   (net 0 "")
@@
     (effects (font (size 0.992 0.992) (thickness 0.1476)))
   )
-  (gr_text "wwavusbepp\nv01 (it wasn't me)" (at 95.1865 118.0465) (layer B.SilkS)
+  (gr_text "diy-wwavusbepp\nv01 (it wasn't me)" (at 95.1865 118.0465) (layer B.SilkS)
     (effects (font (size 1.5 1.5) (thickness 0.3)) (justify left mirror))
   )
